Commit message: Working robotiq 140 gripper

File: urdf/robotiq_arg2f.xacro (robot description, xacro)
@@ -11,5 +11,5 @@
         <origin xyz="0 0 0" rpy="0 0 0" />
         <geometry>
-          <mesh filename="package://robotiq_arg2f_model_visualization/meshes/robotiq_arg2f_base_link_fine.stl" />
+          <mesh filename="package://robotiq_140_description/meshes/robotiq_arg2f_base_link_fine.stl" />
         </geometry>
         <material name="">
@@ -20,5 +20,5 @@
         <origin xyz="0 0 0" rpy="0 0 ${pi / 2}" />
         <geometry>
-          <mesh filename="package://robotiq_arg2f_model_visualization/meshes/robotiq_arg2f_base_link_coarse.stl" />
+          <mesh filename="package://robotiq_140_description/meshes/robotiq_arg2f_base_link_coarse.stl" />
         </geometry>
       </collision>

File: urdf/robotiq_arg2f_140_model.xacro (robot description, xacro)
@@ -1,5 +1,5 @@
 <?xml version="1.0"?>
-<robot name="robotiq_arg2f_140_model" xmlns:xacro="http://ros.org/wiki/xacro">
-  <xacro:include filename="$(find robotiq_arg2f_model_visualization)/urdf/robotiq_arg2f_140_model_macro.xacro" />
+<robot name="robotiq_140_description" xmlns:xacro="http://ros.org/wiki/xacro">
+  <xacro:include filename="$(find robotiq_140_description)/urdf/robotiq_arg2f_140_model_macro.xacro" />
   <xacro:robotiq_arg2f_140 prefix=""/>
 </robot>

File: urdf/robotiq_arg2f_140_model_macro.xacro (robot description, xacro)
@@ -1,5 +1,5 @@
 <?xml version="1.0"?>
 <robot xmlns:xacro="http://ros.org/wiki/xacro">
-  <xacro:include filename="$(find robotiq_arg2f_model_visualization)/urdf/robotiq_arg2f_transmission.xacro" />
+  <xacro:include filename="$(find robotiq_140_description)/urdf/robotiq_arg2f_transmission.xacro" />
   <xacro:macro name="outer_knuckle" params="prefix fingerprefix stroke">
     <link name="${prefix}${fingerprefix}_outer_knuckle">
@@ -18,5 +18,5 @@
         <origin xyz="0 0 0" rpy="0 0 0" />
         <geometry>
-          <mesh filename="package://robotiq_arg2f_model_visualization/meshes/robotiq_arg2f_${stroke}_outer_knuckle.stl" />
+          <mesh filename="package://robotiq_140_description/meshes/robotiq_arg2f_${stroke}_outer_knuckle.stl" />
         </geometry>
         <material name="">
@@ -27,5 +27,5 @@
         <origin xyz="0 0 0" rpy="0 0 0" />
         <geometry>
-          <mesh filename="package://robotiq_arg2f_model_visualization/meshes/robotiq_arg2f_${stroke}_outer_knuckle.stl" />
+          <mesh filename="package://robotiq_140_description/meshes/robotiq_arg2f_${stroke}_outer_knuckle.stl" />
         </geometry>
       </collision>
@@ -48,5 +48,5 @@
         <origin xyz="0 0 0" rpy="0 0 0" />
         <geometry>
-          <mesh filename="package://robotiq_arg2f_model_visualization/meshes/robotiq_arg2f_${stroke}_outer_finger.stl" />
+          <mesh filename="package://robotiq_140_description/meshes/robotiq_arg2f_${stroke}_outer_finger.stl" />
         </geometry>
         <material name="">
@@ -57,5 +57,5 @@
         <origin xyz="0 0 0" rpy="0 0 0" />
         <geometry>
-          <mesh filename="package://robotiq_arg2f_model_visualization/meshes/robotiq_arg2f_${stroke}_outer_finger.stl" />
+          <mesh filename="package://robotiq_140_description/meshes/robotiq_arg2f_${stroke}_outer_finger.stl" />
         </geometry>
       </collision>
@@ -78,5 +78,5 @@
         <origin xyz="0 0 0" rpy="0 0 0" />
         <geometry>
-          <mesh filename="package://robotiq_arg2f_model_visualization/meshes/robotiq_arg2f_${stroke}_inner_knuckle.stl" />
+          <mesh filename="package://robotiq_140_description/meshes/robotiq_arg2f_${stroke}_inner_knuckle.stl" />
         </geometry>
         <material name="">
@@ -87,5 +87,5 @@
         <origin xyz="0 0 0" rpy="0 0 0" />
         <geometry>
-          <mesh filename="package://robotiq_arg2f_model_visualization/meshes/robotiq_arg2f_${stroke}_inner_knuckle.stl" />
+          <mesh filename="package://robotiq_140_description/meshes/robotiq_arg2f_${stroke}_inner_knuckle.stl" />
         </geometry>
       </collision>
@@ -108,5 +108,5 @@
         <origin xyz="0 0 0" rpy="0 0 0" />
         <geometry>
-          <mesh filename="package://robotiq_arg2f_model_visualization/meshes/robotiq_arg2f_${stroke}_inner_finger.stl" />
+          <mesh filename="package://robotiq_140_description/meshes/robotiq_arg2f_${stroke}_inner_finger.stl" />
         </geometry>
         <material name="">
@@ -117,5 +117,5 @@
         <origin xyz="0 0 0" rpy="0 0 0" />
         <geometry>
-          <mesh filename="package://robotiq_arg2f_model_visualization/meshes/robotiq_arg2f_${stroke}_inner_finger.stl" />
+          <mesh filename="package://robotiq_140_description/meshes/robotiq_arg2f_${stroke}_inner_finger.stl" />
         </geometry>
       </collision>
@@ -150,5 +150,5 @@
     </joint>
   </xacro:macro>
-  <xacro:include filename="$(find robotiq_arg2f_model_visualization)/urdf/robotiq_arg2f.xacro" />
+  <xacro:include filename="$(find robotiq_140_description)/urdf/robotiq_arg2f.xacro" />
   <xacro:macro name="finger_joint" params="prefix">
     <joint name="${prefix}finger_joint" type="revolute">

Commit message: Changed names of links and joints to make it work with sara description

File: urdf/robotiq_arg2f.xacro (robot description, xacro)
@@ -1,6 +1,6 @@
 <?xml version="1.0"?>
 <robot xmlns:xacro="http://ros.org/wiki/xacro">
-  <xacro:macro name="robotiq_arg2f_base_link" params="prefix">
-    <link name="${prefix}robotiq_arg2f_base_link">
+  <xacro:macro name="robotiq_arg2f_link" params="prefix">
+    <link name="robotiq_arg2f_link">
       <inertial>
         <origin xyz="8.625E-08 -4.6583E-06 0.03145" rpy="0 0 0" />
@@ -14,5 +14,5 @@
         </geometry>
         <material name="">
-          <color rgba="0.1 0.1 0.1 1" />
+          <color rgba="0.5 0.5 0.5 1" />
         </material>
       </visual>

File: urdf/robotiq_arg2f_140_model_macro.xacro (robot description, xacro)
@@ -133,5 +133,5 @@
     <joint name="${prefix}${fingerprefix}_inner_knuckle_joint" type="revolute">
       <origin xyz="0 ${reflect * -0.0127} 0.06142" rpy="${pi / 2 + .725} 0 ${(reflect - 1) * pi / 2}" />
-      <parent link="${prefix}robotiq_arg2f_base_link" />
+      <parent link="${prefix}robotiq_arg2f_link" />
       <child link="${prefix}${fingerprefix}_inner_knuckle" />
       <axis xyz="1 0 0" />
@@ -154,5 +154,5 @@
     <joint name="${prefix}finger_joint" type="revolute">
       <origin xyz="0 -0.030601 0.054905" rpy="${pi / 2 + .725} 0 0" />
-      <parent link="${prefix}robotiq_arg2f_base_link" />
+      <parent link="${prefix}robotiq_arg2f_link" />
       <child link="${prefix}left_outer_knuckle" />
       <axis xyz="-1 0 0" />
@@ -164,5 +164,5 @@
     <joint name="right_outer_knuckle_joint" type="revolute">
       <origin xyz="0 0.030601 0.054905" rpy="${pi / 2 + .725} 0 ${pi}" />
-      <parent link="${prefix}robotiq_arg2f_base_link" />
+      <parent link="${prefix}robotiq_arg2f_link" />
       <child link="${prefix}right_outer_knuckle" />
       <axis xyz="1 0 0" />
@@ -173,5 +173,5 @@
   </xacro:macro>
   <xacro:macro name="robotiq_arg2f_140" params="prefix">
-    <xacro:robotiq_arg2f_base_link prefix="${prefix}"/>
+    <xacro:robotiq_arg2f_link prefix="${prefix}"/>
     <xacro:finger_links prefix="${prefix}" fingerprefix="left" stroke="140"/>
     <xacro:finger_links prefix="${prefix}" fingerprefix="right" stroke="140"/>

Commit message: fixed bug on gripper

File: urdf/robotiq_arg2f.xacro (robot description, xacro)
@@ -2,5 +2,5 @@
 <robot xmlns:xacro="http://ros.org/wiki/xacro">
   <xacro:macro name="robotiq_arg2f_link" params="prefix">
-    <link name="robotiq_arg2f_link">
+    <link name="${prefix}robotiq_arg2f_link">
       <inertial>
         <origin xyz="8.625E-08 -4.6583E-06 0.03145" rpy="0 0 0" />
