Commit message: fixed another bug

File: urdf/robotiq_arg2f_140_model_macro.xacro (robot description, xacro)
@@ -168,5 +168,5 @@
       <axis xyz="1 0 0" />
       <limit lower="0" upper="0.725" velocity="2.0" effort="1000" />
-    <mimic joint="finger_joint" multiplier="-1" offset="0" />
+    <mimic joint="${prefix}finger_joint" multiplier="-1" offset="0" />
     </joint>
     <xacro:finger_joints prefix="${prefix}" fingerprefix="right" reflect="-1.0"/>
